File: Kicad/Speeduino_UFSC/Speeduino_UFSC.kicad_sch (KiCad schematic)
At the start: 1 part

Commit message: Update Kicad
Other:
- sheet Connector: file connector.sch -> connector.kicad_sch
- sheet Fuel & Ignition: file Fuel_Ignition.sch -> Fuel_Ignition.kicad_sch
- sheet Inputs: file inputs.sch -> inputs.kicad_sch
- sheet Outputs: file outputs.sch -> outputs.kicad_sch
- sheet Power: file power.sch -> power.kicad_sch
- sheet Proto Area: file proto.sch -> proto.kicad_sch
Changed lines of the file:
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@@
 			)
 		)
-		(property "Sheetfile" "inputs.sch"
+		(property "Sheetfile" "inputs.kicad_sch"
 			(at 53.34 192.3546 0)
 			(effects
@@
 			)
 		)
-		(property "Sheetfile" "connector.sch"
+		(property "Sheetfile" "connector.kicad_sch"
 			(at 96.52 191.0846 0)
 			(effects
@@
 			)
 		)
-		(property "Sheetfile" "outputs.sch"
+		(property "Sheetfile" "outputs.kicad_sch"
 			(at 120.65 192.3546 0)
 			(effects
@@
 			)
 		)
-		(property "Sheetfile" "Fuel_Ignition.sch"
+		(property "Sheetfile" "Fuel_Ignition.kicad_sch"
 			(at 26.67 192.3546 0)
 			(effects
@@
 			)
 		)
-		(property "Sheetfile" "proto.sch"
+		(property "Sheetfile" "proto.kicad_sch"
 			(at 139.7 192.3546 0)
 			(effects
@@
 			)
 		)
-		(property "Sheetfile" "power.sch"
+		(property "Sheetfile" "power.kicad_sch"
 			(at 74.93 192.3546 0)
 			(effects
