File: Kicad/Speeduino_UFSC/connector.kicad_sch (KiCad schematic)
At the start: 7 parts, among them J1 Conn_01x02, J3 Conn_02x20_Counter_Clockwise

Commit message: Update Kicad
Parts:
- removed J1: Conn_01x02, TerminalBlock_Phoenix:TerminalBlock_Phoenix_PT-1,5-2-5.0-H_1x02_P5.00mm_Horizontal, symbol Connector_Generic:Conn_01x02
- removed J3: Conn_02x20_Counter_Clockwise, Connector_IDC:IDC-Header_2x20_P2.54mm_Vertical, symbol Connector_Generic:Conn_02x20_Odd_Even
- removed JP12, JP13, JP14, JP15, JP16: SolderJumper_2_Bridged, Jumper:SolderJumper-2_P1.3mm_Bridged_Pad1.0x1.5mm, symbol Jumper:SolderJumper_2_Bridged
- added J1: Conn_02x20_Counter_Clockwise, Connector_IDC:IDC-Header_2x20_P2.54mm_Vertical, symbol Connector_Generic:Conn_02x20_Odd_Even
- added J2: Conn_01x02, TerminalBlock_Phoenix:TerminalBlock_Phoenix_PT-1,5-2-5.0-H_1x02_P5.00mm_Horizontal, symbol Connector_Generic:Conn_01x02
- added JP1, JP2, JP3, JP4, JP5: SolderJumper_2_Bridged, Jumper:SolderJumper-2_P1.3mm_Bridged_Pad1.0x1.5mm, symbol Jumper:SolderJumper_2_Bridged
Connections:
- net 12V-SW: now also J2.2 (Pin_2)
- net BOOST-OUT: now also J1.12 (Pin_12)
- net CAM-IN: now also J1.34 (Pin_34)
- net CLT_Sensor: now also J1.37 (Pin_37)
- net CRANK-IN: now also J1.32 (Pin_32)
- net Clutch_in: now also JP5.1 (A)
- net FAN-OUT: now also JP2.1 (A)
- net FUELPUMP-OUT: now also JP3.1 (A)
- net Flex_Sensor: now also JP1.1 (A)
- net GND: now also J1.17 (Pin_17), J1.19 (Pin_19), J1.23 (Pin_23), J1.36 (Pin_36), J2.1 (Pin_1)
- net HC-1-OUT: now also J1.10 (Pin_10)
- net HC-2-OUT: now also J1.6 (Pin_6)
- net IAT_Sensor: now also J1.39 (Pin_39)
- net IDLE-OUT: now also J1.8 (Pin_8)
- net IGN-1-OUT: now also J1.13 (Pin_13)
- net IGN-2-OUT: now also J1.14 (Pin_14)
- net IGN-3-OUT: now also J1.16 (Pin_16)
- net IGN-4-OUT: now also J1.15 (Pin_15)
- net INJ-1-OUT: now also J1.1 (Pin_1), J1.2 (Pin_2)
- net INJ-2-OUT: now also J1.3 (Pin_3), J1.4 (Pin_4)
- net INJ-3-OUT: now also J1.5 (Pin_5), J1.7 (Pin_7)
- net INJ-4-OUT: now also J1.11 (Pin_11), J1.9 (Pin_9)
- net MAP-EXT: now also J1.21 (Pin_21)
- net O2_Sensor: now also J1.40 (Pin_40)
- net PROTO-1: now also J1.27 (Pin_27), JP1.2 (B)
- net PROTO-2: now also J1.29 (Pin_29), JP2.2 (B)
- net PROTO-3: now also J1.31 (Pin_31), JP3.2 (B)
- net PROTO-4: now also J1.33 (Pin_33), JP4.2 (B)
- net PROTO-5: now also J1.35 (Pin_35), JP5.2 (B)
- net STEP-A1: now also J1.20 (Pin_20)
- net STEP-A2: now also J1.18 (Pin_18)
- net STEP-B1: now also J1.22 (Pin_22)
- net STEP-B2: now also J1.24 (Pin_24)
- net TACHO-OUT: now also JP4.1 (A)
- net TPS_Sensor: now also J1.38 (Pin_38)
- net VDDA: now also J1.25 (Pin_25), J1.26 (Pin_26)
- net VR1-: now also J1.28 (Pin_28)
- net VR2-: now also J1.30 (Pin_30)
