File: Kicad/Speeduino_UFSC/power.kicad_sch (KiCad schematic)
At the start: 12 parts, among them U2 LM2940S-5.0

Commit message: Update Kicad
Parts:
- removed C3: 10uF, Capacitor_THT:CP_Radial_D5.0mm_P2.00mm, symbol Device:CP1
- removed C4, C6: 0.1uF, Capacitor_THT:C_Disc_D5.0mm_W2.5mm_P2.50mm, symbol Device:C
- removed C5: 22uF, Capacitor_THT:C_Disc_D7.5mm_W5.0mm_P5.00mm, symbol Device:C
- removed C7: 47uF, Capacitor_THT:CP_Radial_D8.0mm_P5.00mm, symbol Device:CP1
- removed D4: D_TVS, Diode_THT:D_DO-15_P12.70mm_Horizontal, symbol Device:D_Zener
- removed D6: SB230TA, Diode_THT:D_DO-41_SOD81_P7.62mm_Horizontal, symbol Device:D_Schottky
- removed JP1: Jumper_NO_Small, Connector_PinHeader_2.54mm:PinHeader_1x02_P2.54mm_Vertical, symbol Device:Jumper_NO_Small
- removed R2: 10k, Resistor_THT:R_Axial_DIN0204_L3.6mm_D1.6mm_P5.08mm_Horizontal, symbol Device:R
- removed R6: 120R, Resistor_THT:R_Axial_DIN0204_L3.6mm_D1.6mm_P5.08mm_Horizontal, symbol Device:R
- removed U2: LM2940S-5.0, Package_TO_SOT_THT:TO-220-3_Horizontal_TabDown, symbol Regulator_Linear:LM2937xS
- added C20: 10uF, Capacitor_THT:CP_Radial_D5.0mm_P2.00mm, symbol Device:CP1
- added C21, C23: 0.1uF, Capacitor_THT:C_Disc_D5.0mm_W2.5mm_P2.50mm, symbol Device:C
- added C22: 22uF, Capacitor_THT:C_Disc_D7.5mm_W5.0mm_P5.00mm, symbol Device:C
- added C24: 47uF, Capacitor_THT:CP_Radial_D8.0mm_P5.00mm, symbol Device:CP1
- added D7: D_TVS, Diode_THT:D_DO-15_P12.70mm_Horizontal, symbol Device:D_Zener
- added D8: SB230TA, Diode_THT:D_DO-41_SOD81_P7.62mm_Horizontal, symbol Device:D_Schottky
- added JP11: Jumper_NO_Small, Connector_PinHeader_2.54mm:PinHeader_1x02_P2.54mm_Vertical, symbol Device:Jumper_NO_Small
- added R34: 10k, Resistor_THT:R_Axial_DIN0204_L3.6mm_D1.6mm_P5.08mm_Horizontal, symbol Device:R
- added R35: 120R, Resistor_THT:R_Axial_DIN0204_L3.6mm_D1.6mm_P5.08mm_Horizontal, symbol Device:R
- added U6: LM2940S-5.0, Package_TO_SOT_THT:TO-220-3_Horizontal_TabDown, symbol Regulator_Linear:LM2937xS
Connections:
- net 12V-SW: now also D8.2 (A)
- net GND: now also C20.2, C21.2, C22.2, C23.2, C24.2, D7.2 (A), U6.2 (GND)
- net RESET: now also JP11.2, R34.1
- net VDD: now also C23.1, C24.1, R34.2, R35.2, U6.3 (VO)
- net VRegIn: now also C20.1, C21.1, D7.1 (K), D8.1 (K), U6.1 (VI)
- new net: C22.1, JP11.1, R35.1
