File: Kicad/Speeduino_UFSC_V2/Speeduino_UFSC_V2/power.kicad_sch (KiCad schematic)
At the start: 3 parts, among them U6 LM2940S-5.0

Commit message: Add pdf
Parts:
- U6: footprint Package_TO_SOT_THT:TO-220-3_Horizontal_TabDown -> Package_TO_SOT_SMD:TO-263-3_TabPin2
Changed lines of the file:
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@@
 			)
 		)
-		(property "Footprint" "Package_TO_SOT_THT:TO-220-3_Horizontal_TabDown"
+		(property "Footprint" "Package_TO_SOT_SMD:TO-263-3_TabPin2"
 			(at 142.24 59.055 0)
 			(effects
@@
 			)
 		)
-		(property "Datasheet" ""
+		(property "Datasheet" "http://www.ti.com/lit/ds/symlink/lm2937.pdf"
 			(at 142.24 66.04 0)
 			(effects
@@
 			)
 		)
-		(property "Description" ""
+		(property "Description" "500-mA Low Dropout Regulator, TO-263"
 			(at 142.24 64.77 0)
 			(effects
@@
 			)
 		)
-		(property "Description" ""
+		(property "Description" "Power symbol creates a global label with name \"GND\" , ground"
 			(at 142.24 81.28 0)
 			(effects
@@
 			)
 		)
-		(property "Description" ""
+		(property "Description" "Unpolarized capacitor"
 			(at 120.65 74.93 0)
 			(effects
